File: schematics/40W SMPS/40W SMPS.kicad_pcb (KiCad board)
At the start: 2 copper layers, 70 x 50 mm, 128 parts, among them J1 UJC-HP-3-SMT-TR, J2 Screw_Terminal_01x01, J3 Screw_Terminal_01x01, Q1 NMOS, Q2 NMOS, Q3 NMOS, Q4 NMOS, T1 EFD25_750311594, U2 UCC24612-1DBV, U4 TPS25740RGER, U6 VO617A-3X018T

Commit message: finalised board
Parts:
- added R23: 68k, Resistor_SMD:R_0603_1608Metric, F.Cu at (195.2, 76.0)
- C16: renamed from C28; value 0.01uF -> 10nF
- C17: renamed from C30; value 0.01uF -> 10nF
- C21: renamed from C12; footprint PCM_JLCPCB:C_0603 -> PCM_JLCPCB:C_CASE-A-3216-18(mm)
- C22: renamed from C13; footprint PCM_JLCPCB:C_0603 -> PCM_JLCPCB:C_CASE-A-3216-18(mm)
- C8: renamed from C20; value 2200pF -> 22pF
- D9: renamed from D5; footprint Diode_SMD:Littelfuse_PolyZen-LS -> Package_TO_SOT_SMD:SOT-363_SC-70-6; moved to B.Cu
- R22: renamed from R18; value 760k -> 680k
- U1: value ~ -> UCC28780DR
- U2: renamed from U11; value ~ -> NV6115
- U3: renamed from U8; value ~ -> NV6115
- moved C3 2.73 mm to (174.5, 47.5), turned to 90 degrees
- moved D9 2.32 mm to (216.5, 78.8)
- moved C22 0.56 mm to (225.8, 65.2)
- moved TP12 0.56 mm to (227.8, 66.5)
- moved L2 0.37 mm to (226.7, 69.5)
- moved C21 0.25 mm to (223.5, 65.2)
- renumbered C17 to C1, C7 to C10, C8 to C11, C10 to C12, C9 to C13, C27 to C14, C29 to C15, C16 to C18, C11 to C19, C18 to C2, C15 to C20, C14 to C23, C25 to C24, C38 to C25, C36 to C26, C26 to C27, C21 to C28, C35 to C29, C6 to C3, C39 to C30, C37 to C31, C24 to C32, C23 to C33, C22 to C34, C33 to C35, C32 to C36, C34 to C37, C2 to C5, C19 to C6, C3 to C7, C5 to C9, D4 to D1, D1 to D2, D9 to D3, D2 to D4, D7 to D5, D8 to D7, D3 to D8, J2 to J1, J3 to J2, J1 to J3, JP3 to JP2, JP2 to JP3, Q2 to Q1, Q1 to Q2, R14 to R1, R17 to R10, R3 to R11, R5 to R12, R6 to R13, R4 to R14, R27 to R15, R28 to R16, R10 to R17, R9 to R18, R8 to R19, R12 to R2, R7 to R20, R31 to R21, R19 to R24, R36 to R25, R29 to R26, R32 to R27, R34 to R28, R24 to R29, R11 to R3, R20 to R30, R23 to R31, R35 to R32, R25 to R33, R21 to R34, R26 to R35, R22 to R36, R30 to R37, R37 to R38, R33 to R39, R39 to R4, R13 to R5, R38 to R6, R15 to R7, R2 to R8, R16 to R9, TP3 to TP1, TP22 to TP10, TP10 to TP11, TP18 to TP12, TP19 to TP13, TP20 to TP14, TP21 to TP15, TP11 to TP16, TP16 to TP17, TP12 to TP18, TP17 to TP19, TP4 to TP2, TP13 to TP20, TP14 to TP21, TP15 to TP22, TP5 to TP3, TP6 to TP4, TP7 to TP5, TP2 to TP6, TP8 to TP7, TP1 to TP8, U2 to U4, U6 to U5, U4 to U6
Connections:
- C33 pad 1: Net-(D5-K) (its old number) -> Net-(D9-K)
- C33 pad 2: Net-(D5-common) -> Net-(D9-common)
- C34 pad 2: Net-(D5-common) -> Net-(D9-common)
- D9 pad 1: Net-(D5-common) -> GND2
- D9 pad 2: GND2 -> Net-(D9-K)
- D9 pad 3: Net-(D5-K) (its old number) -> (no net)
- R22 pad 1: Net-(Q3-D) -> Net-(R22-Pad1)
- R30 pad 2: Net-(D5-K) (its old number) -> Net-(D9-K)
- R33 pad 2: Net-(D5-K) (its old number) -> Net-(D9-K)
- R34 pad 1: Net-(D5-common) -> Net-(D9-common)
- R36 pad 2: Net-(D5-common) -> Net-(D9-common)
- R38 pad 1: Net-(D5-common) -> Net-(D9-common)
- R39 pad 1: Net-(D5-common) -> Net-(D9-common)
- U5 pad 2: Net-(D5-K) (its old number) -> Net-(D9-K)
Routing:
- net Net-(D9-common): track 0.00 -> 40.9 mm, vias 0 -> 1
- net Net-(D5-common): track 36.1 -> 0.00 mm
- net Net-(D9-K): track 0.00 -> 20.4 mm, vias 0 -> 1
- net Net-(D5-K) (its old number): track 19.5 -> 0.00 mm
- net /VBUS: track 49.2 -> 51.1 mm, vias 1 -> 3
- net Net-(R22-Pad1): track 0.00 -> 1.52 mm
- net GND2: track 67.1 -> 68.0 mm
- net Net-(Q4-G): track 3.33 -> 3.64 mm, vias 2 -> 0
- removed copper zone on F.Cu, net Net-(DB1-+)
