File: schematics/40W SMPS/40W SMPS.kicad_sch (KiCad schematic)
At the start: 128 parts, among them J1 UJC-HP-3-SMT-TR, J2 Screw_Terminal_01x01, J3 Screw_Terminal_01x01, Q1 NMOS, Q2 NMOS, Q3 NMOS, Q4 NMOS, T1 EFD25_750311594, U2 UCC24612-1DBV, U4 TPS25740RGER, U6 VO617A-3X018T

Commit message: finalised board
Parts:
- added R23: 68k, Resistor_SMD:R_0603_1608Metric, symbol Device:R
- C1: renamed from C17; LCSC (none) -> C14663
- C10: renamed from C7; LCSC (none) -> C64705
- C11: renamed from C8; LCSC (none) -> C64705
- C12: renamed from C10; LCSC (none) -> C86295
- C13: renamed from C9; LCSC (none) -> C86295
- C14: renamed from C27; LCSC (none) -> C14663
- C15: renamed from C29; LCSC (none) -> C14663
- C16: renamed from C28; value 0.01uF -> 10nF; LCSC (none) -> C100042
- C17: renamed from C30; value 0.01uF -> 10nF; LCSC (none) -> C100042
- C18: renamed from C16; LCSC (none) -> C15849
- C19: renamed from C11; LCSC (none) -> C62784
- C2: renamed from C18; LCSC (none) -> C1654
- C20: renamed from C15; LCSC (none) -> C23630
- C21: renamed from C12; footprint PCM_JLCPCB:C_0603 -> PCM_JLCPCB:C_CASE-A-3216-18(mm); LCSC (none) -> C7186
- C22: renamed from C13; footprint PCM_JLCPCB:C_0603 -> PCM_JLCPCB:C_CASE-A-3216-18(mm); LCSC (none) -> C7186
- C23: renamed from C14; LCSC (none) -> C88760
- C24: renamed from C25; LCSC (none) -> C30816
- C25: renamed from C38; LCSC (none) -> C100042
- C26: renamed from C36; LCSC (none) -> C519565
- C27: renamed from C26; LCSC (none) -> C30816
- C28: renamed from C21; LCSC (none) -> C1653
- C29: renamed from C35; LCSC (none) -> C14663
- C3: renamed from C6; LCSC (none) -> C6718369
- C30: renamed from C39; LCSC (none) -> C519565
- C31: renamed from C37; LCSC (none) -> C7419419
- C32: renamed from C24; LCSC (none) -> C1621
- C33: renamed from C23; LCSC (none) -> C882553
- C34: renamed from C22; LCSC (none) -> C100042
- C35: renamed from C33; LCSC (none) -> C14663
- C36: renamed from C32; LCSC (none) -> C14663
- C37: renamed from C34; LCSC (none) -> C64705
- C4: LCSC (none) -> C6718369
- C5: renamed from C2; LCSC (none) -> C14663
- C6: renamed from C19; LCSC (none) -> C1653
- C7: renamed from C3; LCSC (none) -> C14663
- C8: renamed from C20; value 2200pF -> 22pF; LCSC (none) -> C1653
- C9: renamed from C5; LCSC (none) -> C14663
- D1: renamed from D4; LCSC (none) -> C117949
- D2: renamed from D1; LCSC (none) -> C117949
- D3: renamed from D9; LCSC (none) -> C19852660
- D4: renamed from D2; LCSC (none) -> C142698
- D5: renamed from D7; LCSC (none) -> C142698
- D6: LCSC (none) -> C117949
- D7: renamed from D8; LCSC (none) -> C117949
- D8: renamed from D3; LCSC (none) -> C142698
- D9: renamed from D5; footprint Diode_SMD:Littelfuse_PolyZen-LS -> Package_TO_SOT_SMD:SOT-363_SC-70-6; LCSC (none) -> C96225
- F1: digikey (none) -> 5923-RSTA2.5BULK-ND
- J1: renamed from J2; now left out of the parts list
- J2: renamed from J3; now left out of the parts list
- J3: renamed from J1; LCSC (none) -> UJC-HP-3-SMT-TR:CUI_UJC-HP-3-SMT-TR
- JP1, L1, L2, TH1, TP9: now left out of the parts list
- JP2: renamed from JP3; now left out of the parts list
- JP3: renamed from JP2; now left out of the parts list
- Q1: renamed from Q2; LCSC (none) -> C460213
- Q2: renamed from Q1; LCSC (none) -> C2876538
- Q3: LCSC (none) -> C460213
- Q4: LCSC (none) -> C2876538
- R1: renamed from R14; LCSC (none) -> C852877
- R10: renamed from R17; LCSC (none) -> C105578
- R11: renamed from R3; LCSC (none) -> C22548
- R12: renamed from R5; LCSC (none) -> C861855
- R13: renamed from R6; LCSC (none) -> C2906986
- R14: renamed from R4; LCSC (none) -> C2930146
- R15: renamed from R27; LCSC (none) -> C109318
- R16: renamed from R28; LCSC (none) -> C105588
- R17: renamed from R10; LCSC (none) -> C109318
- R18: renamed from R9; LCSC (none) -> C108661
- R19: renamed from R8; LCSC (none) -> C109318
- R2: renamed from R12; LCSC (none) -> C4114738
- R20: renamed from R7; LCSC (none) -> C109318
- R21: renamed from R31; LCSC (none) -> C14675
- R22: renamed from R18; value 760k -> 680k; LCSC (none) -> C25822
- R24: renamed from R19; LCSC (none) -> C2960862
- R25: renamed from R36; LCSC (none) -> C22548
- R26: renamed from R29; LCSC (none) -> C109318
- R27: renamed from R32; LCSC (none) -> C313715
- R28: renamed from R34; LCSC (none) -> C5240695
- R29: renamed from R24; LCSC (none) -> C2906986
- R3: renamed from R11; LCSC (none) -> C2984416
- R30: renamed from R20; LCSC (none) -> C23089
- R31: renamed from R23; LCSC (none) -> C861466
- R32: renamed from R35; LCSC (none) -> C22787
- R33: renamed from R25; LCSC (none) -> C23008
- R34: renamed from R21; LCSC (none) -> C47115979
- R35: renamed from R26; LCSC (none) -> C269902
- R36: renamed from R22; LCSC (none) -> C2906993
- R37: renamed from R30; LCSC (none) -> C2907013
- R38: renamed from R37; LCSC (none) -> C861562
- R39: renamed from R33; LCSC (none) -> C482894
- R5: renamed from R13; LCSC (none) -> C852585
- R7: renamed from R15; LCSC (none) -> C137933
- R8: renamed from R2; LCSC (none) -> C22548
- R9: renamed from R16; LCSC (none) -> C3016242
- T1: LCSC (none) -> C48391662
- TP1: renamed from TP3; now left out of the parts list
- TP10: renamed from TP22; now left out of the parts list
- TP11: renamed from TP10; now left out of the parts list
- TP12: renamed from TP18; now left out of the parts list
- TP13: renamed from TP19; now left out of the parts list
- TP14: renamed from TP20; now left out of the parts list
- TP15: renamed from TP21; now left out of the parts list
- TP16: renamed from TP11; now left out of the parts list
- TP17: renamed from TP16; now left out of the parts list
- TP18: renamed from TP12; now left out of the parts list
- TP19: renamed from TP17; now left out of the parts list
- TP2: renamed from TP4; now left out of the parts list
- TP20: renamed from TP13; now left out of the parts list
- TP21: renamed from TP14; now left out of the parts list
- TP22: renamed from TP15; now left out of the parts list
- TP3: renamed from TP5; now left out of the parts list
- TP4: renamed from TP6; now left out of the parts list
- TP5: renamed from TP7; now left out of the parts list
- TP6: renamed from TP2; now left out of the parts list
- TP7: renamed from TP8; now left out of the parts list
- TP8: renamed from TP1; now left out of the parts list
- U1: value ~ -> UCC28780DR; LCSC (none) -> C2859738
- U2: renamed from U11; value ~ -> NV6115; LCSC (none) -> C2844954
- U3: renamed from U8; value ~ -> NV6115; LCSC (none) -> C2844954
- U4: renamed from U2; LCSC (none) -> C2657796
- U5: renamed from U6; LCSC (none) -> C17317941
- U6: renamed from U4; LCSC (none) -> C544310
- renumbered R39 to R4, R38 to R6
Connections:
- net GND2: now also D9.1 (A); no longer D9.2 (A)
- net at C33.1, R30.2, R33.2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: now also D9.2 (K); no longer D9.3 (K)
- net at C33.2, C34.2, R34.1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: now also D9.6 (common); no longer D9.1 (common)
- net at Q3.1 (D): now also R23.1; no longer R22.1
- new net: R22.1, R23.2
Other:
- moved on the sheet: Q3
